File: Copilot_Lite/Copilot_Lite.kicad_sch (KiCad schematic)
At the start: 14 parts, among them J2 JACK_POWER_IN, J3 USB_POWER_IN, J4 USB_PC, J6 5V_ENABLE, J7 SERIAL_AND_GPIO, J8 JACK_POWER_OUT, J9 USB_POWER_OUT

Commit message: lite: Replaced the old 'uCIme' name by the new 'Copilot' one in the board files.
Signed-off-by: Adrien Ricciardi <aricciardi@baylibre.com>
Other:
- title: uCIme Lite main page -> Copilot Lite main page
Changed lines of the file:
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@@
   (paper "A4")
   (title_block
-    (title "uCIme Lite main page")
+    (title "Copilot Lite main page")
     (date "2023-03-27")
     (company "(C) BayLibre")
@@
     (pin "2")
     (instances
-      (project "uCIme_Lite"
+      (project "Copilot_Lite"
         (path "/6d46d15a-8cd0-4983-b142-8248cafa0b56"
           (reference "D2") (unit 1)
@@
     (pin "S4")
     (instances
-      (project "uCIme_Lite"
+      (project "Copilot_Lite"
         (path "/6d46d15a-8cd0-4983-b142-8248cafa0b56"
           (reference "J8") (unit 1)
@@
     (pin "2")
     (instances
-      (project "uCIme_Lite"
+      (project "Copilot_Lite"
         (path "/6d46d15a-8cd0-4983-b142-8248cafa0b56"
           (reference "R3") (unit 1)
@@
     (pin "1")
     (instances
-      (project "uCIme_Lite"
+      (project "Copilot_Lite"
         (path "/6d46d15a-8cd0-4983-b142-8248cafa0b56"
           (reference "#PWR0104") (unit 1)
@@
     )
     (instances
-      (project "uCIme_Lite"
+      (project "Copilot_Lite"
         (path "/6d46d15a-8cd0-4983-b142-8248cafa0b56"
           (reference "H1") (unit 1)
@@
     (pin "1")
     (instances
-      (project "uCIme_Lite"
+      (project "Copilot_Lite"
         (path "/6d46d15a-8cd0-4983-b142-8248cafa0b56"
           (reference "#PWR0105") (unit 1)
@@
     (pin "1")
     (instances
-      (project "uCIme_Lite"
+      (project "Copilot_Lite"
         (path "/6d46d15a-8cd0-4983-b142-8248cafa0b56"
           (reference "#PWR0108") (unit 1)
@@
     )
     (instances
-      (project "uCIme_Lite"
+      (project "Copilot_Lite"
         (path "/6d46d15a-8cd0-4983-b142-8248cafa0b56"
           (reference "H3") (unit 1)
@@
     (pin "1")
     (instances
-      (project "uCIme_Lite"
+      (project "Copilot_Lite"
         (path "/6d46d15a-8cd0-4983-b142-8248cafa0b56"
           (reference "#PWR07") (unit 1)
@@
     (pin "1")
     (instances
-      (project "uCIme_Lite"
+      (project "Copilot_Lite"
         (path "/6d46d15a-8cd0-4983-b142-8248cafa0b56"
           (reference "#PWR0101") (unit 1)
@@
     (pin "S4")
     (instances
-      (project "uCIme_Lite"
+      (project "Copilot_Lite"
         (path "/6d46d15a-8cd0-4983-b142-8248cafa0b56"
           (reference "J2") (unit 1)
@@
     (pin "A9")
     (instances
-      (project "uCIme_Lite"
+      (project "Copilot_Lite"
         (path "/6d46d15a-8cd0-4983-b142-8248cafa0b56"
           (reference "J3") (unit 1)
@@
     (pin "1")
     (instances
-      (project "uCIme_Lite"
+      (project "Copilot_Lite"
         (path "/6d46d15a-8cd0-4983-b142-8248cafa0b56"
           (reference "#PWR0103") (unit 1)
@@
     (pin "2")
     (instances
-      (project "uCIme_Lite"
+      (project "Copilot_Lite"
         (path "/6d46d15a-8cd0-4983-b142-8248cafa0b56"
           (reference "J6") (unit 1)
@@
     (pin "1")
     (instances
-      (project "uCIme_Lite"
+      (project "Copilot_Lite"
         (path "/6d46d15a-8cd0-4983-b142-8248cafa0b56"
           (reference "#PWR0112") (unit 1)
@@
     (pin "2")
     (instances
-      (project "uCIme_Lite"
+      (project "Copilot_Lite"
         (path "/6d46d15a-8cd0-4983-b142-8248cafa0b56"
           (reference "R4") (unit 1)
@@
     (pin "1")
     (instances
-      (project "uCIme_Lite"
+      (project "Copilot_Lite"
         (path "/6d46d15a-8cd0-4983-b142-8248cafa0b56"
           (reference "#PWR0113") (unit 1)
@@
     (pin "1")
     (instances
-      (project "uCIme_Lite"
+      (project "Copilot_Lite"
         (path "/6d46d15a-8cd0-4983-b142-8248cafa0b56"
           (reference "#PWR06") (unit 1)
@@
     (pin "A9")
     (instances
-      (project "uCIme_Lite"
+      (project "Copilot_Lite"
         (path "/6d46d15a-8cd0-4983-b142-8248cafa0b56"
           (reference "J4") (unit 1)
@@
     )
     (instances
-      (project "uCIme_Lite"
+      (project "Copilot_Lite"
         (path "/6d46d15a-8cd0-4983-b142-8248cafa0b56"
           (reference "H4") (unit 1)
@@
     )
     (instances
-      (project "uCIme_Lite"
+      (project "Copilot_Lite"
         (path "/6d46d15a-8cd0-4983-b142-8248cafa0b56"
           (reference "H2") (unit 1)
@@
     (pin "9")
     (instances
-      (project "uCIme_Lite"
+      (project "Copilot_Lite"
         (path "/6d46d15a-8cd0-4983-b142-8248cafa0b56"
           (reference "J7") (unit 1)
@@
     (pin "1")
     (instances
-      (project "uCIme_Lite"
+      (project "Copilot_Lite"
         (path "/6d46d15a-8cd0-4983-b142-8248cafa0b56"
           (reference "#PWR0110") (unit 1)
@@
     (pin "A9")
     (instances
-      (project "uCIme_Lite"
+      (project "Copilot_Lite"
         (path "/6d46d15a-8cd0-4983-b142-8248cafa0b56"
           (reference "J9") (unit 1)
@@
     (pin "1")
     (instances
-      (project "uCIme_Lite"
+      (project "Copilot_Lite"
         (path "/6d46d15a-8cd0-4983-b142-8248cafa0b56"
           (reference "#PWR0102") (unit 1)
@@
     (pin "1")
     (instances
-      (project "uCIme_Lite"
+      (project "Copilot_Lite"
         (path "/6d46d15a-8cd0-4983-b142-8248cafa0b56"
           (reference "#PWR0109") (unit 1)
@@
     (pin "1")
     (instances
-      (project "uCIme_Lite"
+      (project "Copilot_Lite"
         (path "/6d46d15a-8cd0-4983-b142-8248cafa0b56"
           (reference "#PWR0111") (unit 1)
@@
     )
     (instances
-      (project "uCIme_Lite"
+      (project "Copilot_Lite"
         (path "/6d46d15a-8cd0-4983-b142-8248cafa0b56" (page "3"))
       )
@@
     )
     (instances
-      (project "uCIme_Lite"
+      (project "Copilot_Lite"
         (path "/6d46d15a-8cd0-4983-b142-8248cafa0b56" (page "2"))
       )
