File: Copilot_Lite/Power_Management.kicad_sch (KiCad schematic)
At the start: 21 parts, among them J1 POWER_MODES, Q1 BSS138, Q2 BUK7M27-80EX, Q3 BUK7M27-80EX, Q4 BSS138, U1 LM74502, U2 LM74502

Commit message: lite: Replaced the old 'uCIme' name by the new 'Copilot' one in the board files.
Signed-off-by: Adrien Ricciardi <aricciardi@baylibre.com>
Other:
- title: uCIme Lite power switches -> Copilot Lite power switches
Changed lines of the file:
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@@
   (paper "A4")
   (title_block
-    (title "uCIme Lite power switches")
+    (title "Copilot Lite power switches")
     (date "2023-03-27")
     (company "(C) BayLibre")
@@
     (pin "1")
     (instances
-      (project "uCIme_Lite"
+      (project "Copilot_Lite"
         (path "/6d46d15a-8cd0-4983-b142-8248cafa0b56/b72074d7-db6e-4ce2-896d-216adccf1d19"
           (reference "#PWR0114") (unit 1)
@@
     (pin "1")
     (instances
-      (project "uCIme_Lite"
+      (project "Copilot_Lite"
         (path "/6d46d15a-8cd0-4983-b142-8248cafa0b56/b72074d7-db6e-4ce2-896d-216adccf1d19"
           (reference "#PWR0115") (unit 1)
@@
     (pin "2")
     (instances
-      (project "uCIme_Lite"
+      (project "Copilot_Lite"
         (path "/6d46d15a-8cd0-4983-b142-8248cafa0b56/b72074d7-db6e-4ce2-896d-216adccf1d19"
           (reference "C4") (unit 1)
@@
     (pin "2")
     (instances
-      (project "uCIme_Lite"
+      (project "Copilot_Lite"
         (path "/6d46d15a-8cd0-4983-b142-8248cafa0b56/b72074d7-db6e-4ce2-896d-216adccf1d19"
           (reference "R8") (unit 1)
@@
     (pin "5")
     (instances
-      (project "uCIme_Lite"
+      (project "Copilot_Lite"
         (path "/6d46d15a-8cd0-4983-b142-8248cafa0b56/b72074d7-db6e-4ce2-896d-216adccf1d19"
           (reference "Q3") (unit 1)
@@
     (pin "3")
     (instances
-      (project "uCIme_Lite"
+      (project "Copilot_Lite"
         (path "/6d46d15a-8cd0-4983-b142-8248cafa0b56/b72074d7-db6e-4ce2-896d-216adccf1d19"
           (reference "Q1") (unit 1)
@@
     (pin "1")
     (instances
-      (project "uCIme_Lite"
+      (project "Copilot_Lite"
         (path "/6d46d15a-8cd0-4983-b142-8248cafa0b56/b72074d7-db6e-4ce2-896d-216adccf1d19"
           (reference "#PWR0121") (unit 1)
@@
     (pin "2")
     (instances
-      (project "uCIme_Lite"
+      (project "Copilot_Lite"
         (path "/6d46d15a-8cd0-4983-b142-8248cafa0b56/b72074d7-db6e-4ce2-896d-216adccf1d19"
           (reference "C3") (unit 1)
@@
     (pin "1")
     (instances
-      (project "uCIme_Lite"
+      (project "Copilot_Lite"
         (path "/6d46d15a-8cd0-4983-b142-8248cafa0b56/b72074d7-db6e-4ce2-896d-216adccf1d19"
           (reference "#PWR0116") (unit 1)
@@
     (pin "2")
     (instances
-      (project "uCIme_Lite"
+      (project "Copilot_Lite"
         (path "/6d46d15a-8cd0-4983-b142-8248cafa0b56/b72074d7-db6e-4ce2-896d-216adccf1d19"
           (reference "R1") (unit 1)
@@
     (pin "2")
     (instances
-      (project "uCIme_Lite"
+      (project "Copilot_Lite"
         (path "/6d46d15a-8cd0-4983-b142-8248cafa0b56/b72074d7-db6e-4ce2-896d-216adccf1d19"
           (reference "C1") (unit 1)
@@
     (pin "1")
     (instances
-      (project "uCIme_Lite"
+      (project "Copilot_Lite"
         (path "/6d46d15a-8cd0-4983-b142-8248cafa0b56/b72074d7-db6e-4ce2-896d-216adccf1d19"
           (reference "#PWR0123") (unit 1)
@@
     (pin "8")
     (instances
-      (project "uCIme_Lite"
+      (project "Copilot_Lite"
         (path "/6d46d15a-8cd0-4983-b142-8248cafa0b56/b72074d7-db6e-4ce2-896d-216adccf1d19"
           (reference "U2") (unit 1)
@@
     (pin "2")
     (instances
-      (project "uCIme_Lite"
+      (project "Copilot_Lite"
         (path "/6d46d15a-8cd0-4983-b142-8248cafa0b56/b72074d7-db6e-4ce2-896d-216adccf1d19"
           (reference "D1") (unit 1)
@@
     (pin "2")
     (instances
-      (project "uCIme_Lite"
+      (project "Copilot_Lite"
         (path "/6d46d15a-8cd0-4983-b142-8248cafa0b56/b72074d7-db6e-4ce2-896d-216adccf1d19"
           (reference "D3") (unit 1)
@@
     (pin "1")
     (instances
-      (project "uCIme_Lite"
+      (project "Copilot_Lite"
         (path "/6d46d15a-8cd0-4983-b142-8248cafa0b56/b72074d7-db6e-4ce2-896d-216adccf1d19"
           (reference "#PWR0120") (unit 1)
@@
     (pin "1")
     (instances
-      (project "uCIme_Lite"
+      (project "Copilot_Lite"
         (path "/6d46d15a-8cd0-4983-b142-8248cafa0b56/b72074d7-db6e-4ce2-896d-216adccf1d19"
           (reference "#PWR04") (unit 1)
@@
     (pin "1")
     (instances
-      (project "uCIme_Lite"
+      (project "Copilot_Lite"
         (path "/6d46d15a-8cd0-4983-b142-8248cafa0b56/b72074d7-db6e-4ce2-896d-216adccf1d19"
           (reference "#PWR0118") (unit 1)
@@
     (pin "1")
     (instances
-      (project "uCIme_Lite"
+      (project "Copilot_Lite"
         (path "/6d46d15a-8cd0-4983-b142-8248cafa0b56/b72074d7-db6e-4ce2-896d-216adccf1d19"
           (reference "#PWR02") (unit 1)
@@
     (pin "2")
     (instances
-      (project "uCIme_Lite"
+      (project "Copilot_Lite"
         (path "/6d46d15a-8cd0-4983-b142-8248cafa0b56/b72074d7-db6e-4ce2-896d-216adccf1d19"
           (reference "R2") (unit 1)
@@
     (pin "8")
     (instances
-      (project "uCIme_Lite"
+      (project "Copilot_Lite"
         (path "/6d46d15a-8cd0-4983-b142-8248cafa0b56/b72074d7-db6e-4ce2-896d-216adccf1d19"
           (reference "U1") (unit 1)
@@
     (pin "1")
     (instances
-      (project "uCIme_Lite"
+      (project "Copilot_Lite"
         (path "/6d46d15a-8cd0-4983-b142-8248cafa0b56/b72074d7-db6e-4ce2-896d-216adccf1d19"
           (reference "#PWR0122") (unit 1)
@@
     (pin "1")
     (instances
-      (project "uCIme_Lite"
+      (project "Copilot_Lite"
         (path "/6d46d15a-8cd0-4983-b142-8248cafa0b56/b72074d7-db6e-4ce2-896d-216adccf1d19"
           (reference "#PWR0119") (unit 1)
@@
     (pin "2")
     (instances
-      (project "uCIme_Lite"
+      (project "Copilot_Lite"
         (path "/6d46d15a-8cd0-4983-b142-8248cafa0b56/b72074d7-db6e-4ce2-896d-216adccf1d19"
           (reference "C2") (unit 1)
@@
     (pin "2")
     (instances
-      (project "uCIme_Lite"
+      (project "Copilot_Lite"
         (path "/6d46d15a-8cd0-4983-b142-8248cafa0b56/b72074d7-db6e-4ce2-896d-216adccf1d19"
           (reference "R6") (unit 1)
@@
     (pin "2")
     (instances
-      (project "uCIme_Lite"
+      (project "Copilot_Lite"
         (path "/6d46d15a-8cd0-4983-b142-8248cafa0b56/b72074d7-db6e-4ce2-896d-216adccf1d19"
           (reference "R7") (unit 1)
@@
     (pin "2")
     (instances
-      (project "uCIme_Lite"
+      (project "Copilot_Lite"
         (path "/6d46d15a-8cd0-4983-b142-8248cafa0b56/b72074d7-db6e-4ce2-896d-216adccf1d19"
           (reference "R5") (unit 1)
@@
     (pin "5")
     (instances
-      (project "uCIme_Lite"
+      (project "Copilot_Lite"
         (path "/6d46d15a-8cd0-4983-b142-8248cafa0b56/b72074d7-db6e-4ce2-896d-216adccf1d19"
           (reference "Q2") (unit 1)
@@
     (pin "1")
     (instances
-      (project "uCIme_Lite"
+      (project "Copilot_Lite"
         (path "/6d46d15a-8cd0-4983-b142-8248cafa0b56/b72074d7-db6e-4ce2-896d-216adccf1d19"
           (reference "#PWR08") (unit 1)
@@
     (pin "1")
     (instances
-      (project "uCIme_Lite"
+      (project "Copilot_Lite"
         (path "/6d46d15a-8cd0-4983-b142-8248cafa0b56/b72074d7-db6e-4ce2-896d-216adccf1d19"
           (reference "#PWR05") (unit 1)
@@
     (pin "3")
     (instances
-      (project "uCIme_Lite"
+      (project "Copilot_Lite"
         (path "/6d46d15a-8cd0-4983-b142-8248cafa0b56/b72074d7-db6e-4ce2-896d-216adccf1d19"
           (reference "Q4") (unit 1)
@@
     (pin "1")
     (instances
-      (project "uCIme_Lite"
+      (project "Copilot_Lite"
         (path "/6d46d15a-8cd0-4983-b142-8248cafa0b56/b72074d7-db6e-4ce2-896d-216adccf1d19"
           (reference "#PWR03") (unit 1)
@@
     (pin "2")
     (instances
-      (project "uCIme_Lite"
+      (project "Copilot_Lite"
         (path "/6d46d15a-8cd0-4983-b142-8248cafa0b56/b72074d7-db6e-4ce2-896d-216adccf1d19"
           (reference "R10") (unit 1)
@@
     (pin "2")
     (instances
-      (project "uCIme_Lite"
+      (project "Copilot_Lite"
         (path "/6d46d15a-8cd0-4983-b142-8248cafa0b56/b72074d7-db6e-4ce2-896d-216adccf1d19"
           (reference "R9") (unit 1)
@@
     (pin "6")
     (instances
-      (project "uCIme_Lite"
+      (project "Copilot_Lite"
         (path "/6d46d15a-8cd0-4983-b142-8248cafa0b56/b72074d7-db6e-4ce2-896d-216adccf1d19"
           (reference "J1") (unit 1)
