File: Copilot_Lite/Hardware/Copilot_Lite.kicad_pcb (KiCad board)
At the start: 4 copper layers, 65 x 56 mm, 80 parts, among them J1 POWER_MODES, J11 SERIAL_MODE, J12 SERIAL_VOLTAGE_SELECT, J2 JACK_POWER_IN, J3 USB_POWER_IN, J4 USB_PC, J6 5V_ENABLE, J7 SERIAL_AND_GPIO, J8 JACK_POWER_OUT, J9 USB_POWER_OUT, Q1 BSS138, Q2 BUK7M27-80EX, Q3 BUK7M27-80EX, Q4 BSS138, Q5 BSS138, Q6 BSS138, Q7 BSS138, Q8 BSS138, Q9 BSS138, U1 LM74502, U2 LM74502, U3 AP2204K-ADJ, U4 AP2204K-ADJ, U5 FT230XS, U6 SN74LV1T125, U7 SN74LV1T125, U8 SN74LV1T125, U9 SN74LV1T125

Commit message: Copilot_Lite: Hardware: Convert the schematic and the PCB to KiCad 9
Use the most recent files format, so any future board modification can be
more easily compared with the previous ones.

Signed-off-by: Adrien Ricciardi <aricciardi@baylibre.com>
Parts:
- D1: renamed from D?; value POWER_SWITCH -> JACK_POWER
- D3: renamed from D?; value POWER_SWITCH -> USB_POWER
