File: Copilot_Lite/Hardware/Copilot_Lite.kicad_pcb (KiCad board)
At the start: 4 copper layers, 65 x 56 mm, 80 parts, among them J1 POWER_MODES, J11 SERIAL_MODE, J12 SERIAL_VOLTAGE_SELECT, J2 JACK_POWER_IN, J3 USB_POWER_IN, J4 USB_PC, J6 5V_ENABLE, J7 SERIAL_AND_GPIO, J8 JACK_POWER_OUT, J9 USB_POWER_OUT, Q1 BSS138, Q2 BUK7M27-80EX, Q3 BUK7M27-80EX, Q4 BSS138, Q5 BSS138, Q6 BSS138, Q7 BSS138, Q8 BSS138, Q9 BSS138, U1 LM74502, U2 LM74502, U3 AP2204K-ADJ, U4 AP2204K-ADJ, U5 FT230XS, U6 SN74LV1T125, U7 SN74LV1T125, U8 SN74LV1T125, U9 SN74LV1T125

Commit message: Copilot_Lite: Hardware: Bump the board version to 1.3
Signed-off-by: Adrien Ricciardi <aricciardi@baylibre.com>
Other:
- board text added: "Version 1.3"
- board text removed: "Version 1.2"
Changed lines of the file:
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@@
 	(title_block
 		(title "Copilot Lite")
-		(date "2023-08-25")
-		(rev "1.2")
+		(date "2026-03-02")
+		(rev "1.3")
 		(company "(C) BayLibre")
 	)
@@
 		)
 	)
-	(gr_text "Version 1.2"
+	(gr_text "Version 1.3"
 		(at 110 71.4 0)
 		(layer "F.SilkS")
